File: output_design/ldo_regulator.kicad_pcb (KiCad board)
At the start: 2 copper layers, 150 x 100 mm, 5 parts, among them U1 3.3V

Commit message: feat(components): integrate jlcpcb/lcsc database with 600k+ parts
- Add jlcparts wrapper for parametric search and exact lookup

- Implement automatic catalog download and split-zip extraction

- Map JLC packages to KiCad footprints and symbols automatically

- Unify component database with fallback to built-in catalog

- Add helpers for regulator, mcu, and category-based searches

- Verify 15 tests passing with real manufacturer mpns
Parts:
- C2: value 22uF -> 10uF
- R1: value 330 -> 10k
Changed lines of the file:
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@@
       (effects (font (size 1 1) (thickness 0.15)))
     )
-    (property "Value" "22uF" (at 0 2.5 0) (layer "F.Fab")
+    (property "Value" "10uF" (at 0 2.5 0) (layer "F.Fab")
       (effects (font (size 1 1) (thickness 0.15)))
     )
@@
       (effects (font (size 1 1) (thickness 0.15)))
     )
-    (property "Value" "330" (at 0 2.5 0) (layer "F.Fab")
+    (property "Value" "10k" (at 0 2.5 0) (layer "F.Fab")
       (effects (font (size 1 1) (thickness 0.15)))
     )
