File: output_design/ldo_regulator.kicad_sch (KiCad schematic)
At the start: 5 parts, among them U1 3.3V

Commit message: feat(components): integrate jlcpcb/lcsc database with 600k+ parts
- Add jlcparts wrapper for parametric search and exact lookup

- Implement automatic catalog download and split-zip extraction

- Map JLC packages to KiCad footprints and symbols automatically

- Unify component database with fallback to built-in catalog

- Add helpers for regulator, mcu, and category-based searches

- Verify 15 tests passing with real manufacturer mpns
Parts:
- C2: value 22uF -> 10uF
- R1: value 330 -> 10k
Changed lines of the file:
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@@
   (title_block
     (title "ldo_regulator")
-    (comment 1 "Design a 5V to 3.3V LDO regulator circuit with green LED indicator")
+    (comment 1 "Find a 3.3V LDO 500mA SOT-23")
   )
   (symbol
@@
       (effects (font (size 1.27 1.27)))
     )
-    (property "Value" "22uF" (at 130.00 53.00 0)
+    (property "Value" "10uF" (at 130.00 53.00 0)
       (effects (font (size 1.27 1.27)))
     )
@@
       (effects (font (size 1.27 1.27)))
     )
-    (property "Value" "330" (at 210.00 53.00 0)
+    (property "Value" "10k" (at 210.00 53.00 0)
       (effects (font (size 1.27 1.27)))
     )
